File: window-sensor.kicad_pcb (KiCad board)
At the start: 4 copper layers, 49.7 x 14.5 mm, 24 parts, among them J1 Conn_01x06, U1 NORA-B216-00B, U2 LIS2DTW12TR, U3 SHT4x, U4 TMAG5273, Y1 32.768kHz

Commit message: Finalize PCB before fab
Parts:
- added REF**: KiCad-Logo_5mm_SilkScreen, Symbol:KiCad-Logo_5mm_SilkScreen, B.Cu at (103.8, 64.2)
- added REF**: OSHW-Symbol_6.7x6mm_SilkScreen, Symbol:OSHW-Symbol_6.7x6mm_SilkScreen, B.Cu at (79.5, 63.7)
Other:
- board text added: "https://github.com/usimd/window-sensor, Rev ${REVISION}"
